Commit message: Milestone 4: Gazebo Fortress digital twin, bringup and single-file machine config
- belt_marking_gazebo: world (physics, sensors, overview camera), ros_gz bridges
  (joint commands, QA camera, create/remove/set_pose services), gz_twin_node: laser
  mark decals travel with the belt, cut pieces (with their marks) spawned as dynamic
  bodies and ejected down the chute into the bin, knife/laser head/beam joints animated
- belt_marking_bringup: config/machine.yaml (single source, TODO markers), multi-laser
  overlay, config_loader + stack builder, sim/real/multi_laser_sim launch files
- URDF fixes (unique beam link name, belt strip to conveyor end, centred QA camera)
- docs/images/gazebo_overview.jpg captured from the running simulation

File: ros2_ws/src/belt_marking_description/urdf/belt_marking_machine.urdf.xacro (robot description, xacro)
@@ -12,5 +12,5 @@
   <xacro:arg name="station_offsets" default="0.0"/>        <!-- metres, space separated -->
   <xacro:arg name="knife_offset" default="0.056"/>         <!-- legacy "metalw" = 56 mm -->
-  <xacro:arg name="camera_offset" default="0.030"/>
+  <xacro:arg name="camera_offset" default="0.032"/>
   <xacro:arg name="knife_stroke" default="0.12"/>
   <xacro:arg name="laser_field" default="0.05"/>
@@ -52,8 +52,8 @@
   <xacro:fixed_box name="guide_r" parent="bed" x="0" y="${-belt_w/2 - 0.004}" z="0.02"
                    sx="${bed_len}" sy="0.004" sz="0.01" material="dark" mass="0.3"/>
-  <!-- belt strip on the bed from the entrance to the knife (static visual; the moving
-       belt content - marks, cut pieces - is handled by gz_twin_node / RViz markers) -->
-  <xacro:fixed_box name="belt_strip" parent="base_link" x="${(x_min + knife_x)/2}" y="0"
-                   z="${belt_z - 0.002}" sx="${knife_x - x_min}" sy="${belt_w}" sz="0.002"
+  <!-- belt strip on the bed (static visual). The moving belt content (laser marks, cut
+       pieces) is spawned and moved by gz_twin_node in Gazebo and by rviz_markers_node. -->
+  <xacro:fixed_box name="belt_strip" parent="base_link" x="${(x_min + x_max)/2}" y="0"
+                   z="${belt_z - 0.002}" sx="${x_max - x_min}" sy="${belt_w}" sz="0.002"
                    material="belt_black" mass="0.05" collision="false"/>
   <!-- supply reel -->
@@ -103,5 +103,5 @@
     <joint name="qa_camera_joint" type="fixed">
       <parent link="base_link"/><child link="qa_camera_link"/>
-      <origin xyz="${cam_x} ${-0.035} ${belt_z + 0.09}" rpy="0 ${pi/2} 0"/>
+      <origin xyz="${cam_x} 0 ${belt_z + 0.08}" rpy="0 ${pi/2} 0"/>
     </joint>
     <link name="qa_camera_optical_frame"/>

File: ros2_ws/src/belt_marking_description/urdf/gazebo.xacro (robot description, xacro)
@@ -27,5 +27,5 @@
       <gazebo reference="laser_${idx}_carriage"><gravity>false</gravity></gazebo>
       <gazebo reference="laser_${idx}_head"><gravity>false</gravity></gazebo>
-      <gazebo reference="laser_${idx}_beam"><gravity>false</gravity></gazebo>
+      <gazebo reference="laser_${idx}_beam_link"><gravity>false</gravity></gazebo>
       <xacro:gz_station idx="${idx + 1}" n="${n}"/>
     </xacro:if>
@@ -41,5 +41,5 @@
         <topic>/qa_camera/image_raw</topic>
         <camera>
-          <horizontal_fov>0.62</horizontal_fov>
+          <horizontal_fov>0.8</horizontal_fov>
           <image><width>640</width><height>480</height><format>R8G8B8</format></image>
           <clip><near>0.02</near><far>2.0</far></clip>

File: ros2_ws/src/belt_marking_description/urdf/macros.xacro (robot description, xacro)
@@ -113,5 +113,5 @@
     </joint>
     <!-- beam (96 mm): hidden inside the head at 0, bottom touches the belt at 0.13 -->
-    <link name="laser_${idx}_beam">
+    <link name="laser_${idx}_beam_link">
       <visual>
         <origin xyz="0 0 -0.048"/>
@@ -123,5 +123,5 @@
     <joint name="laser_${idx}_beam" type="prismatic">
       <parent link="laser_${idx}_head"/>
-      <child link="laser_${idx}_beam"/>
+      <child link="laser_${idx}_beam_link"/>
       <origin xyz="0 0 0.06"/>
       <axis xyz="0 0 -1"/>
